File: em_hardware/power.kicad_sch (KiCad schematic)
At the start: 23 parts, among them J1 USB_C_Receptacle_USB2.0_16P, U3 BQ24074RGT, U5 CH340N

Commit message: done the power
sensors next
Parts:
- added C8, C9: 10uf, symbol Device:C
- added D2: RED_LED, symbol Device:LED
- added D3: GREEN_LED, symbol Device:LED
- added R13, R14: 22, symbol Device:R
- added TP4: D+_TP, symbol Connector:TestPoint
- added TP5: D-_TP, symbol Connector:TestPoint
- added TP6: GND_TP, symbol Connector:TestPoint
- added TP7: 3V3_TP, symbol Connector:TestPoint
- added U2: TPD2EUSB30, Package_TO_SOT_SMD:SOT-23-6, symbol Power_Protection:TPD2EUSB30
- added U6: AP2112K-3.3, Package_TO_SOT_SMD:SOT-23-5, symbol Regulator_Linear:AP2112K-3.3
- R8, R9: value 100k -> 2.2k
- TP2: value CHG_TP -> 5V_TP
- TP3: value PGOOD_TP -> PWR_TP
Connections:
- net 3v3: now also C9.1, TP7.1, U6.5 (VOUT)
- net D+: now also R13.2, TP4.1; no longer J1.A6 (D+), J1.B6 (D+)
- net D-: now also R14.2, TP5.1; no longer J1.A7 (D-), J1.B7 (D-)
- net GND: now also C8.2, C9.2, TP6.1, U2.3 (GND), U6.2 (GND)
- net PWR_RAIL: now also TP3.1, C8.1, U6.1 (VIN), U6.3 (EN)
- net USB_5V_PROTECTED: now also TP2.1
- removed net CHG: R9.1, TP2.1, U3.7 (~{PGOOD})
- removed net PGOOD: R8.1, TP3.1, U3.9 (~{CHG})
- new net: D3.2 (A), R9.1
- new net: J1.A6 (D+), J1.B6 (D+), R13.1, U2.1 (D+)
- new net: D3.1 (K), U3.7 (~{PGOOD})
- new net: D2.1 (K), U3.9 (~{CHG})
- new net: D2.2 (A), R8.1
- new net: J1.A7 (D-), J1.B7 (D-), R14.1, U2.2 (D-)
Other:
- moved on the sheet: C5, J1

Commit message: making this a lot smaller and adding modules
Parts:
- added C12: 1uf, Capacitor_SMD:C_0201_0603Metric_Pad0.64x0.40mm_HandSolder, symbol Device:C
- added R17: 10k, Resistor_SMD:R_0201_0603Metric_Pad0.64x0.40mm_HandSolder, symbol Device:R
- added U7: LC709203FQH-01TWG, Package_DFN_QFN:WDFN-8-1EP_4x3mm_P0.65mm_EP2.4x1.8mm_ThermalVias, symbol Battery_Management:LC709203FQH-01TWG
- C1, C2, C3, C4, C5, C8, C9: footprint (none) -> Capacitor_SMD:C_0201_0603Metric_Pad0.64x0.40mm_HandSolder
- D2, D3: footprint (none) -> LED_SMD:LED_0201_0603Metric_Pad0.64x0.40mm_HandSolder
- F1: footprint (none) -> Fuse:Fuse_0603_1608Metric
- J1: footprint Connector_USB:USB_C_Receptacle_Amphenol_12401948E412A -> Connector_USB:USB_C_Receptacle_GCT_USB4105-xx-A_16P_TopMnt_Horizontal
- R1, R10, R13, R14, R2, R3, R4, R5, R6, R7, R8, R9: footprint (none) -> Resistor_SMD:R_0201_0603Metric_Pad0.64x0.40mm_HandSolder
- TP1, TP2, TP3, TP4, TP5, TP6, TP7: footprint (none) -> TestPoint:TestPoint_Pad_1.0x1.0mm
Connections:
- net BAT+: now also C12.2, U7.3 (V_{DD})
- net GND: now also C12.1, R17.2, U7.1 (TEST), U7.2 (V_{SS})
- net RX0: now also U5.6 (TXD); no longer U5.7 (RXD)
- net TX0: now also U5.7 (RXD); no longer U5.6 (TXD)
- new net LC7_INT: R17.1, U7.4 (~{ALARMB})
- new net SCL: U7.8 (SCL)
- new net SDA: U7.7 (SDA)
- no-connect marks 2 -> 4
Other:
- note added: "3v3 regulator"
- note added: "POWER MONITOR"
