File: em_hardware/em_hardware.kicad_sch (KiCad schematic)
At the start: 7 parts, among them SW1 SW_Push, SW2 SW_Push, U1 ESP32-WROOM-32

Commit message: done the power
sensors next
Other:
- moved on the sheet: C6, C7, R11, R12, SW1, SW2, U1

Commit message: making this a lot smaller and adding modules
Parts:
- added C10, C11: 0.1uf, Capacitor_SMD:C_0201_0603Metric_Pad0.64x0.40mm_HandSolder, symbol Device:C
- added C13: 1uf, Capacitor_SMD:C_0201_0603Metric_Pad0.64x0.40mm_HandSolder, symbol Device:C
- added J2, J3: Conn_01x04_Socket, Connector_PinSocket_2.54mm:PinSocket_1x04_P2.54mm_Vertical_SMD_Pin1Left, symbol Connector:Conn_01x04_Socket
- added U4: BMI160, Package_LGA:Bosch_LGA-14_3x2.5mm_P0.5mm, symbol Sensor_Motion:BMI160
- BOOT_IO0: renamed from SW2; footprint (none) -> Button_Switch_SMD:SW_SPST_B3U-1000P-B
- C6: value C -> 0.1uf; footprint (none) -> Capacitor_SMD:C_0201_0603Metric_Pad0.64x0.40mm_HandSolder
- C7: value C -> 1uf; footprint (none) -> Capacitor_SMD:C_0201_0603Metric_Pad0.64x0.40mm_HandSolder
- EN1: renamed from SW1; footprint (none) -> Button_Switch_SMD:SW_SPST_B3U-1000P-B
- R11, R12: footprint (none) -> Resistor_SMD:R_0201_0603Metric_Pad0.64x0.40mm_HandSolder
Connections:
- net 3v3: now also C10.1, C11.2, J2.1 (Pin_1), U4.1 (SDO), U4.12 (CSB), U4.5 (VDDIO), U4.8 (VDD)
- net GND: now also C10.2, C11.1, C13.2, J2.4 (Pin_4), J3.1 (Pin_1), U4.6 (GNDIO), U4.7 (GND)
- net at EN1.2, R11.1, U1.3 (EN): now also C13.1
- net BMI_INT2: now reaches U1.10 (IO25)
- net BMI_INT2: now also U4.9 (INT2)
- net MAX_INT: now reaches U1.11 (IO26)
- net MAX_INT: now also J3.4 (Pin_4)
- net LC7_INT: now reaches U1.28 (IO17)
- net SCL: now reaches U1.33 (IO21)
- net SCL: now also J2.3 (Pin_3), U4.13 (SCx)
- net SDA: now reaches U1.36 (IO22)
- net SDA: now also J2.2 (Pin_2), U4.14 (SDx)
- no-connect marks 0 -> 7
Other:
- moved on the sheet: C7

Commit message: almost done the PCB
Parts:
- removed J2, J3: Conn_01x04_Socket, Connector_PinSocket_2.54mm:PinSocket_1x04_P2.54mm_Vertical_SMD_Pin1Left, symbol Connector:Conn_01x04_Socket
- added J2, J3: Conn_01x06_Pin, Connector_PinSocket_2.54mm:PinSocket_1x06_P2.54mm_Vertical_SMD_Pin1Left, symbol Connector:Conn_01x06_Pin
- added J4: Conn_01x02_Socket, Connector_JST:JST_PH_S2B-PH-K_1x02_P2.00mm_Horizontal, symbol Connector:Conn_01x02_Socket
Connections:
- net GND: now also J4.2 (Pin_2)
- new net BAT+: J4.1 (Pin_1)

Commit message: PCB DESIGN IS DONE
Susie is alive
Parts:
- J2: footprint Connector_PinSocket_2.54mm:PinSocket_1x06_P2.54mm_Vertical_SMD_Pin1Left -> Connector_PinHeader_2.54mm:PinHeader_1x06_P2.54mm_Vertical
- J3: footprint Connector_PinSocket_2.54mm:PinSocket_1x06_P2.54mm_Vertical_SMD_Pin1Left -> Connector_JST:JST_SH_SM06B-SRSS-TB_1x06-1MP_P1.00mm_Horizontal
Connections:
- net 3v3: now also J2.1 (Pin_1), J3.1 (Pin_1)
- net BMI_INT2: no longer U1.10 (IO25)
- net GND: now also J2.6 (Pin_6), J3.6 (Pin_6)
- net SCL: now also J2.2 (Pin_2), J3.2 (Pin_2)
- net SDA: now also J2.3 (Pin_3), J3.3 (Pin_3)
- net INT: now reaches J2.4 (Pin_4)
- net INT: now also J3.4 (Pin_4), U1.37 (IO23)
- net AUX: now reaches J2.5 (Pin_5)
- net AUX: now also J3.5 (Pin_5), U1.31 (IO19)
- net MAX_INT: no longer names the net of U1.11 (IO26)
- no-connect marks 7 -> 5
Other:
- moved on the sheet: J3
