File: em_hardware/em_hardware.kicad_pcb (KiCad board)
At the start: 2 copper layers, 51 parts, among them J1 USB_C_Receptacle_USB2.0_16P, J2 Conn_01x04_Socket, J3 Conn_01x04_Socket, U1 ESP32-WROOM-32, U2 TPD2EUSB30, U3 BQ24074RGT, U4 BMI160, U5 CH340N, U6 AP2112K-3.3, U7 LC709203FQH-01TWG

Commit message: almost done the PCB
Parts:
- C12, R17, U7: moved to B.Cu
- TP1: moved to F.Cu
- moved C12 135.9 mm to (217.6, 81.0), turned to 90 degrees
- moved U7 135.4 mm to (217.0, 76.6)
- moved R17 134.5 mm to (216.4, 81.0), turned to -90 degrees
- moved C8 128.9 mm to (206.3, 67.0), turned to 90 degrees
- moved U6 127.9 mm to (209.1, 66.5)
- moved C9 125.8 mm to (206.3, 65.0), turned to -90 degrees
- moved TP3 118.9 mm to (197.8, 81.4), turned to 180 degrees
- moved TP7 117.5 mm to (200.8, 81.4), turned to 180 degrees
- moved TP1 42.9 mm to (213.6, 70.4)
- moved R10 31.6 mm to (199.2, 67.4), turned to 90 degrees
- moved R7 29.5 mm to (198.2, 67.4), turned to 90 degrees
- moved C4 29.4 mm to (198.8, 74.6), turned to 90 degrees
- moved R4 29.1 mm to (205.6, 71.4), turned to 0 degrees
- moved R8 28.9 mm to (203.0, 74.6), turned to 90 degrees
- moved R9 28.7 mm to (205.6, 75.8)
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Routing:
- net GND: track 95.0 -> 170.1 mm, vias 1 -> 6
- net 3v3: track 49.6 -> 91.7 mm, vias 1 -> 4
- net PWR_RAIL: track 0.00 -> 37.9 mm, vias 0 -> 1
- net BAT+: track 0.00 -> 33.2 mm, vias 0 -> 3
- net SDA: track 0.00 -> 31.3 mm, vias 0 -> 1
- net SCL: track 0.00 -> 28.0 mm, vias 0 -> 1
- net LC7_INT: track 0.00 -> 27.4 mm, vias 0 -> 1
- net D-: track 0.00 -> 23.9 mm, vias 0 -> 3
- net USB_5V_PROTECTED: track 2.67 -> 26.5 mm, vias 0 -> 2
- net D+: track 0.00 -> 18.9 mm, vias 0 -> 3
- net Net-(D3-K): track 0.00 -> 5.43 mm
- net Net-(U3-ISET): track 0.00 -> 3.09 mm
- net Net-(U3-EN1): track 0.00 -> 2.82 mm
- net Net-(U3-EN2): track 0.00 -> 2.62 mm
- net Net-(U3-TS): track 0.00 -> 2.27 mm
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Other:
- board outline added: 38 x 46 mm

Commit message: idk
Parts:
- added J4: Conn_01x02_Socket, Connector_JST:JST_PH_S2B-PH-K_1x02_P2.00mm_Horizontal, F.Cu at (222.3, 79.9)
Routing:
- net GND: track 170.1 -> 179.2 mm
- net BAT+: track 33.2 -> 37.9 mm
Other:
- board size 38 x 46 mm -> 42 x 46 mm

Commit message: added gnd shielding
Parts:
- removed C10, C11: 0.1uf, Capacitor_SMD:C_0201_0603Metric_Pad0.64x0.40mm_HandSolder
- removed U4: BMI160, Package_LGA:Bosch_LGA-14_3x2.5mm_P0.5mm
- J2: value Conn_01x04_Socket -> Conn_01x06_Pin; footprint Connector_PinHeader_2.54mm:PinHeader_1x04_P2.54mm_Vertical -> Connector_PinHeader_2.54mm:PinHeader_1x06_P2.54mm_Vertical; moved to F.Cu
- J3: value Conn_01x04_Socket -> Conn_01x06_Pin; footprint Connector_PinHeader_2.54mm:PinHeader_1x04_P2.54mm_Vertical -> Connector_JST:JST_SH_SM06B-SRSS-TB_1x06-1MP_P1.00mm_Horizontal; moved to F.Cu
- moved J3 130.8 mm to (227.0, 50.0), turned to 90 degrees
- moved J2 118.0 mm to (224.0, 61.9)
Connections:
- J2 pad 2: SDA -> SCL
- J2 pad 3: SCL -> SDA
- J2 pad 4: GND -> INT
- J3 pad 1: GND -> 3v3
- J3 pad 2: unconnected-(J3-Pin_2-Pad2) -> SCL
- J3 pad 3: unconnected-(J3-Pin_3-Pad3) -> SDA
- J3 pad 4: MAX_INT -> INT
- U1 pad 10: BMI_INT2 -> unconnected-(U1-IO25-Pad10)
- U1 pad 11: MAX_INT -> unconnected-(U1-IO26-Pad11)
- U1 pad 31: unconnected-(U1-IO19-Pad31) -> AUX
- U1 pad 37: unconnected-(U1-IO23-Pad37) -> INT
Routing:
- net AUX: track 0.00 -> 46.4 mm, vias 0 -> 2
- net INT: track 0.00 -> 30.4 mm
- net 3v3: track 91.7 -> 121.1 mm, vias 4 -> 5
- net GND: track 179.2 -> 190.6 mm
- net SDA: track 31.3 -> 40.2 mm, vias 1 -> 2
- net SCL: track 28.0 -> 35.0 mm, vias 1 -> 2
- added copper zone on B.Cu, net GND
- added copper zone on F.Cu, net GND
Other:
- outline, holes or cut-outs redrawn
- board text added: "PROJECT: SUSIE DEVELOPED BY ASHER MOBUOGWU MAY 2026"
