File: em_hardware/Suzie/Suzie.kicad_sch (KiCad schematic)
At the start: 0 parts

Commit message: hardware stuff
I need to make the USB module
Parts:
- added C1, C2: 100nf, symbol Device:C
- added C10, C9: C, symbol Device:C
- added C3, C4: 4.7uf, symbol Device:C
- added C5: 10uf, symbol Device:C
- added C6: 0.1uf, symbol Device:C
- added C7: 1uf, symbol Device:C
- added R1, R2: 4.7k, symbol Device:R
- added R3, R5, R6, R9: 10k, symbol Device:R
- added R7, R8: 22, symbol Device:R
- added SW1, SW2: SW_Push, Battery:BatteryHolder_Bulgin_BX0034_1xAAA, symbol Switch:SW_Push
- added U1: ESP32-C3-WROOM-02, RF_Module:ESP32-S2-WROVER, symbol RF_Module:ESP32-C3-WROOM-02
- added U2: BMI160, Package_LGA:Bosch_LGA-14_3x2.5mm_P0.5mm, symbol Sensor_Motion:BMI160
- added U3: MCP1826S, Package_TO_SOT_SMD:SOT-223-3_TabPin2, symbol Regulator_Linear:MCP1826S
Connections:
- new net: R9.1, U1.16 (IO2)
- new net: R5.1, U1.7 (IO8)
- new net: R6.2, SW2.2, U1.8 (IO9)
- new net 3V3: C1.1, C2.1, C5.1, C6.1, R1.1, R2.1, R3.1, R5.2, R6.1, R9.2, U1.1 (3V3), U2.1 (SDO), U2.12 (CSB), U2.5 (VDDIO), U2.8 (VDD)
- new net 3v3: C4.1, U3.3 (VO)
- new net 5v: C3.2, U3.1 (VI)
- new net D+: R8.2, U1.14 (IO19)
- new net D-: R7.2, U1.13 (IO18)
- new net EN: C7.1, R3.2, SW1.1, U1.2 (EN)
- new net GND: C1.2, C10.2, C2.2, C3.1, C4.2, C5.2, C6.2, C7.2, C9.2, SW1.2, SW2.1, U1.19 (GND), U1.9 (GND), U2.6 (GNDIO), U2.7 (GND), U3.2 (GND)
- new net RX: U1.11 (IO20/RXD)
- new net SCL: R1.2, U2.13 (SCx)
- new net SDA: R2.2, U2.14 (SDx)
- new net TX: U1.12 (IO21/TXD)
- new net USB_D+: C10.1, R8.1
- new net USB_D-: C9.1, R7.1
- new net bmi160_int1: U2.4 (INT1)
- new net bmi160_int2: U2.9 (INT2)
Other:
- note added: "BMI160 circuit"
- note added: "power supply for esp32"
- note added: "voltage regulator"

Commit message: removed the USB data lines
it is for charging only
Parts:
- added J1: USB_C_Receptacle_USB2.0_16P, Connector_USB:USB_C_Receptacle_Amphenol_12401948E412A, symbol Connector:USB_C_Receptacle_USB2.0_16P
- added R10, R4: 5.1k, symbol Device:R
Connections:
- net 3v3 is gone; now on net 3V3: C4.1, U3.3 (VO)
- net GND: now also J1.A1 (GND), J1.A12 (GND), J1.B1 (GND), J1.B12 (GND), J1.SH (SHIELD), R10.2, R4.2
- net USB_D+: now also J1.A6 (D+), J1.B6 (D+)
- net USB_D-: now also J1.A7 (D-), J1.B7 (D-)
- net 5v renamed 5V
- new net: J1.A5 (CC1), R10.1
- new net: J1.B5 (CC2), R4.1
- new net VBUS: J1.A4 (VBUS), J1.A9 (VBUS), J1.B4 (VBUS), J1.B9 (VBUS)
- no-connect marks 0 -> 2
Other:
- moved on the sheet: C7, R3, SW1

Commit message: tbc
Parts:
- removed C10, C9: C, symbol Device:C
- removed C4: 4.7uf, symbol Device:C
- removed U3: MCP1826S, Package_TO_SOT_SMD:SOT-223-3_TabPin2, symbol Regulator_Linear:MCP1826S
- added C8: 10uf, symbol Device:C
- added Q2: 2N3906, Package_TO_SOT_THT:TO-92_Inline, symbol Transistor_BJT:2N3906
- added U4: TLV75533PDBV, Package_TO_SOT_SMD:SOT-23-5, symbol Regulator_Linear:TLV75533PDBV
- C3: value 4.7uf -> 1uf
- R7, R8: value 22 -> 1k
Connections:
- net 3V3: now also C8.1, U4.5 (OUT)
- net GND: now also C8.2, Q2.3 (C), U4.2 (GND)
- net VBUS: now also R7.2
- net 5V renamed VBAT
- net VBAT: now also R8.2, U4.1 (IN)
- net D+: no longer names the net of U1.14 (IO19)
- net D+: no longer R8.2
- net D-: no longer names the net of U1.13 (IO18)
- net D-: no longer R7.2
- removed net USB_D+: J1.A6 (D+), J1.B6 (D+), R8.1
- removed net USB_D-: J1.A7 (D-), J1.B7 (D-), R7.1
- new net: Q2.2 (B), R7.1
- new net Suzie_EN: Q2.1 (E), R8.1, U4.3 (EN)
- no-connect marks 2 -> 4
Other:
- note removed: "voltage regulator"
